File: RelayTimer/RelayTimer.kicad_pcb (KiCad board)
At the start: 2 copper layers, 89 x 74.3 mm, 20 parts, among them J1 Jack-DC, J2 Relay_Con, Q1 2N3904, U1 ATtiny85-20P

Commit message: minor update to KiCad project
Parts:
- moved R6 2.44 mm to (195.3, 101.1), turned to 90 degrees
Connections:
- R6 pad 1: PB3_PULLUP -> +5V
- R6 pad 2: +5V -> PB3_PULLUP
Other:
- board text added: "Press 'FUNCTION' to add time Press both buttons to reset time"
- board text removed: "Press 'FUNCTION' to add time Hold 'FUNCTION' to reset time"

Commit message: added small reset button to schematic
Parts:
- added SW1: SW_Push, Button_Switch_THT:SW_PUSH_6mm, F.Cu at (145.4, 139.2)
Connections:
- U1 pad 1: unconnected-(U1-~{RESET}/PB5-Pad1) -> Net-(U1-~{RESET}/PB5)
Routing:
- net Net-(U1-~{RESET}/PB5): track 0.00 -> 7.79 mm
Other:
- board text added: "Reset"

Commit message: forgot to update the revision number
Other:
- board text added: "rev2.2"
- board text removed: "rev2.0"
Changed lines of the file:
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@@
 		(fp_arc
 			(start 64.20104 22.49932)
-			(mid 64.054473 22.853115)
+			(mid 64.054479 22.85315)
 			(end 63.70066 22.9997)
 			(stroke
@@
 		)
 	)
-	(gr_text "rev2.0"
+	(gr_text "rev2.2"
 		(at 156 136.95 20)
 		(layer "F.SilkS")

Commit message: fixed small issue and updated board
Parts:
- removed R4, R5: 1k, Resistor_THT:R_Axial_DIN0204_L3.6mm_D1.6mm_P2.54mm_Vertical
- R6, R7: footprint Resistor_THT:R_Axial_DIN0204_L3.6mm_D1.6mm_P2.54mm_Vertical -> Resistor_THT:R_Axial_DIN0204_L3.6mm_D1.6mm_P7.62mm_Horizontal
- moved R6 2.49 mm to (195.2, 98.6), turned to -90 degrees
- moved R7 2.49 mm to (192.8, 98.6), turned to -90 degrees
- moved C4 2.05 mm to (174.0, 76.2), turned to 0 degrees
- moved C3 2.05 mm to (178.8, 76.2), turned to 0 degrees
Connections:
- FUNCTION1 pad 2: Net-(FUNCTION1-Pad2) -> PB4_PULLUP
- R6 pad 1: +5V -> PB3_PULLUP
- R6 pad 2: PB3_PULLUP -> +5V
- R7 pad 1: +5V -> PB4_PULLUP
- R7 pad 2: PB4_PULLUP -> +5V
- START/STOP1 pad 2: Net-(R5-Pad1) -> PB3_PULLUP
Routing:
- net Net-(FUNCTION1-Pad2): track 34.6 -> 0.00 mm
- net Net-(R5-Pad1): track 19.4 -> 0.00 mm
- net PB3_PULLUP: track 93.3 -> 108.4 mm
- net Net-(U1-~{RESET}/PB5): track 7.79 -> 14.3 mm
- net +5V: track 180.1 -> 175.3 mm
- net SDA: track 92.4 -> 93.7 mm
- net SCL: track 96.1 -> 97.2 mm
- net PB4_PULLUP: track 109.1 -> 108.2 mm
Other:
- board text added: "Hold 'FUNCTION' to add time Press both buttons to reset time"
- board text added: "rev2.3"
- board text removed: "Press 'FUNCTION' to add time Press both buttons to reset time"
- board text removed: "rev2.2"
